File: airquality.sch (KiCad schematic (older format))
At the start: 18 parts, among them J1 MHZ19, J2 Conn_02x10_Odd_Even, J3 Conn_02x10_Odd_Even, J4 Conn_01x04_Female, J5 Conn_01x04_Male, J6 Conn_01x04_Female, J7 Conn_01x04_Male, J8 Conn_01x04_Male, U1 DS18B20, U2 PMS7003, U3 RFM95W-868S2, U4 DS18B20, U5 DS18B20

Commit message: rev2
Parts:
- removed AE1: Antenna, RF_Antenna:Texas_SWRA416_868MHz_915MHz, symbol Device:Antenna
- removed C3: 100nF, Capacitor_SMD:C_0805_2012Metric_Pad1.15x1.40mm_HandSolder, symbol Device:C
- removed J8: Conn_01x04_Male, Connector_JST:JST_PH_S4B-PH-K_1x04_P2.00mm_Horizontal, symbol Connector:Conn_01x04_Male
- removed U3: RFM95W-868S2, RFM95W-915S2:XCVR_RFM95W-915S2, symbol RFM95W-915S2:RFM95W-915S2
- removed U5: DS18B20, Package_TO_SOT_THT:TO-92_Inline, symbol Sensor_Temperature:DS18B20
- added C1: 100nF, Capacitor_SMD:C_0805_2012Metric_Pad1.15x1.40mm_HandSolder, symbol Device:C
- added D1: SK6812, LED_SMD:LED_SK6812_PLCC4_5.0x5.0mm_P3.2mm, symbol LED:SK6812
- added H1, H2: MountingHole, MountingHole:MountingHole_4.3mm_M4, symbol Mechanical:MountingHole
- added H3, H4: MountingHole, parts_models:keyhole, symbol Mechanical:MountingHole
- added H5, H6, H7, H8: MountingHole, MountingHole:MountingHole_3.2mm_M3, symbol Mechanical:MountingHole
- added J10, J11, J13, J14, J15, J16, J2, J22, J25, J3, J4, J5, J6, J7, J8, J9: Conn_01x01_Male, Connector_PinHeader_2.54mm:PinHeader_1x01_P2.54mm_Vertical, symbol Connector:Conn_01x01_Male
- added J23, J24: Conn_01x04_Female, Connector_PinSocket_2.54mm:PinSocket_1x04_P2.54mm_Vertical, symbol Connector:Conn_01x04_Female
- added Q1: BSS138, Package_TO_SOT_SMD:SOT-23, symbol Transistor_FET:BSS138
- added R1, R2, R3: 4k7, Resistor_SMD:R_0805_2012Metric_Pad1.15x1.40mm_HandSolder, symbol Device:R
- added SW1: SW_Push, Button_Switch_SMD:SW_SPST_TL3342, symbol Switch:SW_Push
- renumbered C1 to C5, C2 to C6, J2 to J1, J3 to J12, J1 to J17, J4 to J18, J6 to J19, J5 to J20, J7 to J21, R1 to R4, U2 to U1, U1 to U2, U4 to U3
Connections:
- net 1wire: now also J22.1 (Pin_1)
- net 3.3V: now also J13.1 (Pin_1), J23.2 (Pin_2), J24.1 (Pin_1), Q1.1 (G), R1.1, R2.1
- net 5V: now also J17.1 (VIN), C1.1, D1.3 (VDD), J16.1 (Pin_1), R3.1; no longer J17.3 (V0)
- net GND: now also C1.2, D1.1 (VSS), J14.1 (Pin_1), J15.1 (Pin_1), J23.1 (Pin_1), J24.2 (Pin_2), SW1.2
- net I2C_SCL: now also J23.3 (Pin_3), J24.4 (Pin_4)
- net I2C_SDA: now also J23.4 (Pin_4), J24.3 (Pin_3)
- net IO14: now also J8.1 (Pin_1)
- net IO15: now also R2.2, SW1.1
- net IO16: now also J4.1 (Pin_1)
- net IO17: now also J3.1 (Pin_1)
- net IO18: now also J7.1 (Pin_1)
- net IO19: now also J5.1 (Pin_1)
- net IO26: now also Q1.2 (S), R1.2
- net IO27: now also J2.1 (Pin_1)
- net IO33: now also J11.1 (Pin_1)
- net IO34: now also J10.1 (Pin_1)
- net IO35: now also J9.1 (Pin_1)
- net IO5: now also J6.1 (Pin_1)
- net NC: no longer names the net of J1.16 (Pin_16)
- net NC: no longer J1.4 (Pin_4)
- new net: D1.2 (DIN), Q1.3 (D), R3.2
- new net: D1.4 (DOUT), J25.1 (Pin_1)
- no-connect marks 0 -> 2
